File: nfc-pcb/nfc-pcb.kicad_pcb (KiCad board)
At the start: 2 copper layers, 5 parts, among them U1 NT3H1101W0FHKH

Commit message: update
Parts:
- moved C1 6.22 mm to (124.0, 81.1)
- moved D1 6.22 mm to (123.9, 75.8)
- moved R1 6.22 mm to (119.3, 78.1)
- moved L1 6.22 mm to (100.0, 55.0)
- moved U1 6.22 mm to (124.0, 86.2)
Other:
- board outline added: 55 x 42.5 mm
Changed lines of the file:
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@@
 	(footprint "Resistor_SMD:R_1206_3216Metric"
 		(layer "F.Cu")
-		(at 125 80.5 90)
+		(at 119.258516 78.1 90)
 		(descr "Resistor SMD 1206 (3216 Metric), square (rectangular) end terminal, IPC_7351 nominal, (Body size source: IPC-SM-782 page 72, https://www.pcb-3d.com/wordpress/wp-content/uploads/ipc-sm-782a_amendment_1_and_2.pdf), generated with kicad-footprint-generator")
 		(tags "resistor")
@@
 	(footprint "easyeda2kicad:XQFN-8_L1.6-W1.6-P0.50-BR"
 		(layer "F.Cu")
-		(at 129.75 88.6 90)
+		(at 124.008516 86.2 90)
 		(property "Reference" "U1"
 			(at 0 -4.6 90)
@@
 	(footprint "Capacitor_SMD:C_1206_3216Metric"
 		(layer "F.Cu")
-		(at 129.725 83.5)
+		(at 123.983516 81.1)
 		(descr "Capacitor SMD 1206 (3216 Metric), square (rectangular) end terminal, IPC_7351 nominal, (Body size source: IPC-SM-782 page 76, https://www.pcb-3d.com/wordpress/wp-content/uploads/ipc-sm-782a_amendment_1_and_2.pdf), generated with kicad-footprint-generator")
 		(tags "capacitor")
@@
 	(footprint "LED_SMD:LED_1206_3216Metric"
 		(layer "F.Cu")
-		(at 129.65 78.25 180)
+		(at 123.908516 75.85 180)
 		(descr "LED SMD 1206 (3216 Metric), square (rectangular) end terminal, IPC_7351 nominal, (Body size source: http://www.tortai-tech.com/upload/download/2011102023233369053.pdf), generated with kicad-footprint-generator")
 		(tags "LED")
@@
 	(footprint "nfc_ant:antenna-nfc"
 		(layer "F.Cu")
-		(at 105.741484 57.4)
+		(at 100 55)
 		(property "Reference" "L1"
 			(at 25 18.5 0)
@@
 		)
 	)
-	(segment
-		(start 131.2 83.5)
-		(end 129.65 85.05)
+	(gr_line
+		(start 152.5 92.5)
+		(end 152.5 55)
+		(stroke
+			(width 0.05)
+			(type default)
+		)
+		(layer "Edge.Cuts")
+	)
+	(gr_arc
+		(start 100 95)
+		(mid 98.232233 94.267767)
+		(end 97.5 92.5)
+		(stroke
+			(width 0.05)
+			(type default)
+		)
+		(layer "Edge.Cuts")
+	)
+	(gr_arc
+		(start 152.5 92.5)
+		(mid 151.767767 94.267767)
+		(end 150 95)
+		(stroke
+			(width 0.05)
+			(type default)
+		)
+		(layer "Edge.Cuts")
+	)
+	(gr_arc
+		(start 97.5 55)
+		(mid 98.232233 53.232233)
+		(end 100 52.5)
+		(stroke
+			(width 0.05)
+			(type default)
+		)
+		(layer "Edge.Cuts")
+	)
+	(gr_line
+		(start 100 95)
+		(end 150 95)
+		(stroke
+			(width 0.05)
+			(type default)
+		)
+		(layer "Edge.Cuts")
+	)
+	(gr_line
+		(start 97.5 55)
+		(end 97.5 92.5)
+		(stroke
+			(width 0.05)
+			(type default)
+		)
+		(layer "Edge.Cuts")
+	)
+	(gr_line
+		(start 150 52.5)
+		(end 100 52.5)
+		(stroke
+			(width 0.05)
+			(type default)
+		)
+		(layer "Edge.Cuts")
+	)
+	(gr_arc
+		(start 150 52.5)
+		(mid 151.767767 53.232233)
+		(end 152.5 55)
+		(stroke
+			(width 0.05)
+			(type default)
+		)
+		(layer "Edge.Cuts")
+	)
+	(segment
+		(start 125.458516 81.1)
+		(end 123.908516 82.65)
 		(width 0.2)
 		(layer "F.Cu")
@@
 	)
 	(segment
-		(start 129.65 85.05)
-		(end 129.65 87.498529)
+		(start 123.908516 82.65)
+		(end 123.908516 85.098529)
 		(width 0.2)
 		(layer "F.Cu")
@@
 	)
 	(segment
-		(start 129.75 87.598529)
-		(end 129.75 87.95)
+		(start 124.008516 85.198529)
+		(end 124.008516 85.55)
 		(width 0.2)
 		(layer "F.Cu")
@@
 	)
 	(segment
-		(start 129.65 87.498529)
-		(end 129.75 87.598529)
+		(start 123.908516 85.098529)
+		(end 124.008516 85.198529)
 		(width 0.2)
 		(layer "F.Cu")
@@
 	)
 	(segment
-		(start 131.2 78.4)
-		(end 131.05 78.25)
+		(start 125.458516 76)
+		(end 125.308516 75.85)
 		(width 0.2)
 		(layer "F.Cu")
@@
 	)
 	(segment
-		(start 131.2 83.5)
-		(end 131.2 78.4)
+		(start 125.458516 81.1)
+		(end 125.458516 76)
 		(width 0.2)
 		(layer "F.Cu")
@@
 	)
 	(segment
-		(start 130.25 89.25)
-		(end 129.75 89.25)
+		(start 124.508516 86.85)
+		(end 124.008516 86.85)
 		(width 0.2)
 		(layer "F.Cu")
@@
 	)
 	(segment
-		(start 128.25 89.25)
-		(end 128.8 89.8)
+		(start 122.508516 86.85)
+		(end 123.058516 87.4)
 		(width 0.2)
 		(layer "F.Cu")
@@
 	)
 	(segment
-		(start 125 81.9625)
-		(end 126.7125 81.9625)
+		(start 119.258516 79.5625)
+		(end 120.971016 79.5625)
 		(width 0.2)
 		(layer "F.Cu")
@@
 	)
 	(segment
-		(start 128.25 83.5)
-		(end 128.25 89.25)
+		(start 122.508516 81.1)
+		(end 122.508516 86.85)
 		(width 0.2)
 		(layer "F.Cu")
@@
 	)
 	(segment
-		(start 126.7125 81.9625)
-		(end 128.25 83.5)
+		(start 120.971016 79.5625)
+		(end 122.508516 81.1)
 		(width 0.2)
 		(layer "F.Cu")
@@
 	)
 	(segment
-		(start 129.7 89.8)
-		(end 129.75 89.75)
+		(start 123.958516 87.4)
+		(end 124.008516 87.35)
 		(width 0.2)
 		(layer "F.Cu")
@@
 	)
 	(segment
-		(start 128.8 89.8)
-		(end 129.7 89.8)
+		(start 123.058516 87.4)
+		(end 123.958516 87.4)
 		(width 0.2)
 		(layer "F.Cu")
@@
 	)
 	(segment
-		(start 129.75 89.75)
-		(end 129.75 89.25)
+		(start 124.008516 87.35)
+		(end 124.008516 86.85)
 		(width 0.2)
 		(layer "F.Cu")
@@
 	)
 	(segment
-		(start 125.7875 78.25)
-		(end 125 79.0375)
+		(start 120.046016 75.85)
+		(end 119.258516 76.6375)
 		(width 0.2)
 		(layer "F.Cu")
@@
 	)
 	(segment
-		(start 128.25 78.25)
-		(end 125.7875 78.25)
+		(start 122.508516 75.85)
+		(end 120.046016 75.85)
 		(width 0.2)
 		(layer "F.Cu")
@@
 	)
 	(segment
-		(start 130.35 88.6)
-		(end 130.45 88.6)
+		(start 124.608516 86.2)
+		(end 124.708516 86.2)
 		(width 0.2)
 		(layer "F.Cu")
@@
 	)
 	(segment
-		(start 130.45 88.6)
-		(end 131.232968 89.382968)
+		(start 124.708516 86.2)
+		(end 125.491484 86.982968)
 		(width 0.2)
 		(layer "F.Cu")
@@
 	)
 	(segment
-		(start 131.232968 89.382968)
-		(end 131.232968 91.85)
+		(start 125.491484 86.982968)
+		(end 125.491484 89.45)
 		(width 0.2)
 		(layer "F.Cu")
@@
 	)
 	(segment
-		(start 130.25 87.25)
-		(end 130.25 87.95)
+		(start 124.508516 84.85)
+		(end 124.508516 85.55)
 		(width 0.2)
 		(layer "F.Cu")
@@
 	)
 	(via
-		(at 130.25 87.25)
+		(at 124.508516 84.85)
 		(size 0.6)
 		(drill 0.3)
@@
 	)
 	(segment
-		(start 130.25 90.75)
-		(end 130.25 87.25)
+		(start 124.508516 88.35)
+		(end 124.508516 84.85)
 		(width 0.2)
 		(layer "B.Cu")
@@
 	)
 	(segment
-		(start 130.25 94.25)
-		(end 130.25 90.75)
+		(start 124.508516 91.85)
+		(end 124.508516 88.35)
 		(width 0.2)
 		(layer "B.Cu")
@@
 	)
 	(segment
-		(start 130.25 90.75)
-		(end 130.25 90.5)
+		(start 124.508516 88.35)
+		(end 124.508516 88.1)
 		(width 0.2)
 		(layer "B.Cu")
